File: uSDXproto.kicad_sch (KiCad schematic)
At the start: 25 parts, among them J101 Conn_Coaxial, J102 Mike / Key 3.5mm, J103 Headphones 3.5mm, J104 10 pin IDC female, Q101 2N7000, Q102 2N7000, Q103 2N7000, SW101 RotaryEncoder_Switch, SW102 Menu, SW103 Exit

Commit message: update git schematics
Parts:
- added J101: Conn_Coaxial_Power, symbol Connector:Conn_Coaxial_Power
- renumbered C103 to C102, C102 to C103, J101 to J102, J102 to J103, J103 to J104, J104 to J105, L103 to L101, L101 to L102, L102 to L103
Connections:
- net +12V: now also J101.1 (In)
- net GND: now also J101.2 (Ext)
- net RxAnt: no longer C104.1, L101.2, L102.1, Q101.3 (D), Q102.3 (D), Q103.3 (D)
- new net: C104.1, L101.2, L102.1, Q101.3 (D), Q102.3 (D), Q103.3 (D)
Other:
- moved on the sheet: C101, C102, C103, C104, C105, CE101, J102, L101, L102, L103, Q101, Q102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
