File: Processor.kicad_sch (KiCad schematic)
At the start: 21 parts, among them J201 ISP, J202 LCD-4bit, U201 LM78L05_TO92, U202 ATmega328P, Y201 20mhz

Commit message: update kicad schematics
Connections:
- net Si5351-SDA: no longer J202.4 (Pin_4)
- net at U202.9 (PD5): now also J202.4 (Pin_4)
- new net: U202.21 (GND), U202.5 (GND)
- no-connect marks 4 -> 3
Other:
- note added: "LCD D4"
- note added: "LCD D5"
- note added: "LCD D6"
- note added: "LCD D7"
- note added: "LCD E"
- note added: "LCD RS"
Changed lines of the file:
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@@
   (junction (at 154.94 31.75) (diameter 0) (color 0 0 0 0)
-  )
-  (junction (at 196.85 91.44) (diameter 0) (color 0 0 0 0)
   )
   (junction (at 129.54 49.53) (diameter 0) (color 0 0 0 0)
@@
   (no_connect (at 90.17 78.74))
   (no_connect (at 97.79 68.58))
-  (no_connect (at 142.24 114.3))
   (wire (pts (xy 154.94 31.75) (xy 182.88 31.75))
     (stroke (width 0) (type default) (color 0 0 0 0))
@@
     (stroke (width 0) (type default) (color 0 0 0 0))
   )
-  (wire (pts (xy 196.85 91.44) (xy 196.85 107.95))
-    (stroke (width 0) (type default) (color 0 0 0 0))
-  )
   (wire (pts (xy 142.24 137.16) (xy 205.74 137.16))
     (stroke (width 0) (type default) (color 0 0 0 0))
@@
     (stroke (width 0) (type default) (color 0 0 0 0))
   )
-  (wire (pts (xy 142.24 91.44) (xy 196.85 91.44))
-    (stroke (width 0) (type default) (color 0 0 0 0))
-  )
   (wire (pts (xy 100.33 106.68) (xy 100.33 109.22))
     (stroke (width 0) (type default) (color 0 0 0 0))
@@
     (stroke (width 0) (type default) (color 0 0 0 0))
   )
+  (wire (pts (xy 151.13 114.3) (xy 151.13 125.73))
+    (stroke (width 0) (type default) (color 0 0 0 0))
+  )
   (wire (pts (xy 142.24 58.42) (xy 152.4 58.42))
     (stroke (width 0) (type default) (color 0 0 0 0))
@@
     (stroke (width 0) (type default) (color 0 0 0 0))
   )
+  (wire (pts (xy 151.13 125.73) (xy 196.85 125.73))
+    (stroke (width 0) (type default) (color 0 0 0 0))
+  )
   (wire (pts (xy 52.07 41.91) (xy 64.77 41.91))
     (stroke (width 0) (type default) (color 0 0 0 0))
@@
     (stroke (width 0) (type default) (color 0 0 0 0))
   )
+  (wire (pts (xy 142.24 114.3) (xy 151.13 114.3))
+    (stroke (width 0) (type default) (color 0 0 0 0))
+  )
   (wire (pts (xy 95.25 68.58) (xy 95.25 69.85))
     (stroke (width 0) (type default) (color 0 0 0 0))
@@
     (stroke (width 0) (type default) (color 0 0 0 0))
   )
-  (wire (pts (xy 196.85 91.44) (xy 205.74 91.44))
+  (wire (pts (xy 142.24 91.44) (xy 205.74 91.44))
     (stroke (width 0) (type default) (color 0 0 0 0))
   )
@@
     (stroke (width 0) (type default) (color 0 0 0 0))
   )
+  (wire (pts (xy 196.85 125.73) (xy 196.85 107.95))
+    (stroke (width 0) (type default) (color 0 0 0 0))
+  )
   (wire (pts (xy 189.23 77.47) (xy 189.23 105.41))
     (stroke (width 0) (type default) (color 0 0 0 0))
@@
     (stroke (width 0) (type default) (color 0 0 0 0))
   )
+  (text "LCD D6" (at 144.78 106.68 0)
+    (effects (font (size 1.27 1.27)) (justify left bottom))
+  )
+  (text "LCD RS" (at 144.78 114.3 0)
+    (effects (font (size 1.27 1.27)) (justify left bottom))
+  )
+  (text "LCD D7" (at 144.78 109.22 0)
+    (effects (font (size 1.27 1.27)) (justify left bottom))
+  )
+  (text "LCD D4" (at 144.78 101.6 0)
+    (effects (font (size 1.27 1.27)) (justify left bottom))
+  )
+  (text "LCD E" (at 144.78 111.76 0)
+    (effects (font (size 1.27 1.27)) (justify left bottom))
+  )
+  (text "LCD D5" (at 144.78 104.14 0)
+    (effects (font (size 1.27 1.27)) (justify left bottom))
+  )
   (global_label "AFout" (shape input) (at 213.36 53.34 0) (fields_autoplaced)
