File: uSDX_RF.kicad_sch (KiCad schematic)
At the start: 42 parts, among them Q301 2N7000, U301 LM4562, U302 FST3253 or SN74CBT3253(c), U303 Si5351A-B-GT, U304 74ACT00, U305 LM78L05_TO92, U306 7hACT00, Y301 27mhz

Commit message: update kicad schematics
Parts:
- added unit 4 of U304
- renumbered C308 to C307, C307 to C308
Connections:
- net 5Vrf: now also R305.2; no longer C307.1, C313.2, R309.2, U301.1
- net GND: now also C307.1, U301.1, U304.12, U304.13
- new net: C313.2, R309.2
- no-connect marks 0 -> 2
Other:
- moved on the sheet: C307, C308
